File: GP_SUB.kicad_sch (KiCad schematic)
At the start: 34 parts, among them J13 Conn_01x10, J14 Conn_01x10, J32 Conn_01x02, J5 Conn_02x10_Odd_Even, U1 TPS76333, U2 TXB0104RUT, U5 TXB0104RUT

Commit message: Add files via upload
Parts:
- added R91: 0R, Resistor_SMD:R_0603_1608Metric, symbol Device:R_Small
Connections:
- net GP_EN: now also R91.2
- net TP12_Pin8: now also U5.7 (B4); no longer U2.8 (B3)
- net TP15_Pin12: now also U2.8 (B3); no longer U5.7 (B4)
- net TP16_Pin16: now also U2.9 (B2); no longer U5.8 (B3)
- net TP8_Pin13: now also U5.8 (B3); no longer U2.9 (B2)
- net VBUS: now also R91.1
- net at R19.1: now also U5.4 (A3); no longer U2.3 (A2)
- net at R14.1: now also U2.3 (A2); no longer U5.4 (A3)
- net at U5.5 (A4): now also R18.1; no longer R13.1
- net at U2.4 (A3): now also R13.1; no longer R18.1
Other:
- moved on the sheet: J13, J14, J32, J5, R13, R14, R15, R16, R17, R18, R19, R20
