File: MCU.kicad_pcb (KiCad board)
At the start: 4 copper layers, 110.3 x 102.2 mm, 58 parts, among them J1 F31L-1A7H1-11030, J13 Conn_01x10, J14 Conn_01x10, J17 Conn_02x30_Counter_Clockwise, J2 F31L-1A7H1-11030, J3 F31L-1A7H1-11030, J32 Conn_01x02, J4 Conn_02x30_Counter_Clockwise, J5 Conn_02x10_Odd_Even, J6 Conn_01x02, U1 TPS76333, U2 TXB0104RUT, U3 TPS76333, U4 TPS76333, U5 TXB0104RUT

Commit message: Add files via upload
Parts:
- added C15: 100nF, Capacitor_SMD:C_0402_1005Metric, F.Cu at (111.5, 114.3)
- added C18: 100nF, Capacitor_SMD:C_0402_1005Metric, F.Cu at (111.2, 120.7)
- added C19: 100nF, Capacitor_SMD:C_0402_1005Metric, F.Cu at (109.5, 113.5)
- added C20: 100nF, Capacitor_SMD:C_0402_1005Metric, F.Cu at (109.2, 119.8)
- added C21: 1uF, Capacitor_SMD:C_0603_1608Metric, F.Cu at (113.3, 106.1)
- added C22: 4.7uF, Capacitor_SMD:C_0603_1608Metric, F.Cu at (107.1, 107.3)
- added C23: 100nF, Capacitor_SMD:C_0402_1005Metric, F.Cu at (159.7, 73.4)
- added C24: 100nF, Capacitor_SMD:C_0402_1005Metric, F.Cu at (160.0, 67.0)
- added C25: 100nF, Capacitor_SMD:C_0402_1005Metric, F.Cu at (161.7, 74.2)
- added C26: 100nF, Capacitor_SMD:C_0402_1005Metric, F.Cu at (162.0, 67.9)
- added C27: 1uF, Capacitor_SMD:C_0603_1608Metric, F.Cu at (157.9, 81.6)
- added C28: 4.7uF, Capacitor_SMD:C_0603_1608Metric, F.Cu at (164.1, 80.4)
- added C29: 100nF, Capacitor_SMD:C_0402_1005Metric, F.Cu at (159.4, 108.2)
- added C30: 100nF, Capacitor_SMD:C_0402_1005Metric, F.Cu at (159.7, 101.8)
- added C31: 100nF, Capacitor_SMD:C_0402_1005Metric, F.Cu at (161.4, 109.0)
- added C32: 100nF, Capacitor_SMD:C_0402_1005Metric, F.Cu at (161.7, 102.7)
- added C33: 1uF, Capacitor_SMD:C_0603_1608Metric, F.Cu at (157.6, 116.4)
- added C34: 4.7uF, Capacitor_SMD:C_0603_1608Metric, F.Cu at (163.8, 115.2)
- added D4: LED, LED_SMD:LED_0805_2012Metric, F.Cu at (111.2, 108.5)
- added D5: LED, LED_SMD:LED_0805_2012Metric, F.Cu at (160.0, 79.2)
- added D6: LED, LED_SMD:LED_0805_2012Metric, F.Cu at (159.8, 114.0)
- added J10: Conn_02x10_Odd_Even, Connector_PinHeader_2.54mm:PinHeader_2x10_P2.54mm_Vertical, F.Cu at (87.2, 123.9)
- added J11: Conn_01x10, Connector_PinSocket_2.54mm:PinSocket_1x10_P2.54mm_Vertical, F.Cu at (176.8, 85.2)
- added J12: Conn_01x10, Connector_PinSocket_2.54mm:PinSocket_1x10_P2.54mm_Vertical, F.Cu at (169.2, 85.2)
- added J15: Conn_01x02, Connector_PinHeader_2.54mm:PinHeader_1x02_P2.54mm_Vertical, F.Cu at (183.9, 90.4)
- added J16: Conn_02x10_Odd_Even, Connector_PinHeader_2.54mm:PinHeader_2x10_P2.54mm_Vertical, F.Cu at (183.9, 63.8)
- added J18: Conn_01x10, Connector_PinSocket_2.54mm:PinSocket_1x10_P2.54mm_Vertical, F.Cu at (176.6, 120.1)
- added J19: Conn_01x10, Connector_PinSocket_2.54mm:PinSocket_1x10_P2.54mm_Vertical, F.Cu at (168.9, 120.1)
- added J20: Conn_01x02, Connector_PinHeader_2.54mm:PinHeader_1x02_P2.54mm_Vertical, F.Cu at (183.7, 125.2)
- added J21: Conn_02x10_Odd_Even, Connector_PinHeader_2.54mm:PinHeader_2x10_P2.54mm_Vertical, F.Cu at (183.7, 98.6)
- added J7: Conn_01x10, Connector_PinSocket_2.54mm:PinSocket_1x10_P2.54mm_Vertical, F.Cu at (94.3, 102.4)
- added J8: Conn_01x10, Connector_PinSocket_2.54mm:PinSocket_1x10_P2.54mm_Vertical, F.Cu at (102.0, 102.4)
- added J9: Conn_01x02, Connector_PinHeader_2.54mm:PinHeader_1x02_P2.54mm_Vertical, F.Cu at (87.2, 97.3)
- added R21: 0R, Resistor_SMD:R_0201_0603Metric, F.Cu at (107.0, 114.1)
- added R22: 0R, Resistor_SMD:R_0201_0603Metric, F.Cu at (107.0, 114.9)
- added R23: 0R, Resistor_SMD:R_0201_0603Metric, F.Cu at (106.9, 115.7)
- added R24: 0R, Resistor_SMD:R_0201_0603Metric, F.Cu at (106.9, 116.5)
- added R25: 0R, Resistor_SMD:R_0201_0603Metric, F.Cu at (106.7, 120.3)
- added R26: 0R, Resistor_SMD:R_0201_0603Metric, F.Cu at (106.7, 121.2)
- added R27: 0R, Resistor_SMD:R_0201_0603Metric, F.Cu at (106.8, 122.0)
- added R28: 0R, Resistor_SMD:R_0201_0603Metric, F.Cu at (106.8, 122.9)
- added R29: 4k7, Resistor_SMD:R_0603_1608Metric, F.Cu at (114.1, 103.7)
- added R30: 9k1, Resistor_SMD:R_0603_1608Metric, F.Cu at (112.6, 103.7)
- added R31: 1R, Resistor_SMD:R_0603_1608Metric, F.Cu at (107.1, 108.8)
- added R41: 1k, Resistor_SMD:R_0603_1608Metric, F.Cu at (109.4, 108.3)
- added R44: 0R, Resistor_SMD:R_0201_0603Metric, F.Cu at (164.2, 73.6)
- added R47: 0R, Resistor_SMD:R_0201_0603Metric, F.Cu at (164.2, 72.8)
- added R50: 0R, Resistor_SMD:R_0201_0603Metric, F.Cu at (164.3, 72.0)
- added R52: 0R, Resistor_SMD:R_0201_0603Metric, F.Cu at (164.3, 71.2)
- added R53: 0R, Resistor_SMD:R_0201_0603Metric, F.Cu at (164.4, 67.4)
- added R54: 0R, Resistor_SMD:R_0201_0603Metric, F.Cu at (164.4, 66.5)
- added R55: 0R, Resistor_SMD:R_0201_0603Metric, F.Cu at (164.4, 65.7)
- added R56: 0R, Resistor_SMD:R_0201_0603Metric, F.Cu at (164.4, 64.8)
- added R57: 4k7, Resistor_SMD:R_0603_1608Metric, F.Cu at (157.1, 84.0)
- added R58: 9k1, Resistor_SMD:R_0603_1608Metric, F.Cu at (158.6, 84.0)
- added R59: 1R, Resistor_SMD:R_0603_1608Metric, F.Cu at (164.1, 78.9)
- added R68: 1k, Resistor_SMD:R_0603_1608Metric, F.Cu at (161.8, 79.4)
- added R69: 0R, Resistor_SMD:R_0201_0603Metric, F.Cu at (163.9, 108.4)
- added R70: 0R, Resistor_SMD:R_0201_0603Metric, F.Cu at (163.9, 107.6)
- added R71: 0R, Resistor_SMD:R_0201_0603Metric, F.Cu at (164.0, 106.8)
- added R72: 0R, Resistor_SMD:R_0201_0603Metric, F.Cu at (164.0, 106.0)
- added R73: 0R, Resistor_SMD:R_0201_0603Metric, F.Cu at (164.2, 102.2)
- added R74: 0R, Resistor_SMD:R_0201_0603Metric, F.Cu at (164.2, 101.3)
- added R75: 0R, Resistor_SMD:R_0201_0603Metric, F.Cu at (164.1, 100.5)
- added R76: 0R, Resistor_SMD:R_0201_0603Metric, F.Cu at (164.1, 99.6)
- added R77: 4k7, Resistor_SMD:R_0603_1608Metric, F.Cu at (156.9, 118.8)
- added R78: 9k1, Resistor_SMD:R_0603_1608Metric, F.Cu at (158.4, 118.8)
- added R79: 1R, Resistor_SMD:R_0603_1608Metric, F.Cu at (163.8, 113.7)
- added R88: 1k, Resistor_SMD:R_0603_1608Metric, F.Cu at (161.5, 114.2)
- added R89: 1R, Resistor_SMD:R_0603_1608Metric, F.Cu at (64.0, 46.0)
- added R90: 1R, Resistor_SMD:R_0603_1608Metric, F.Cu at (64.0, 48.5)
- added R91: 0R, Resistor_SMD:R_0603_1608Metric, F.Cu at (70.0, 46.0)
- added R92: 0R, Resistor_SMD:R_0603_1608Metric, F.Cu at (70.0, 55.0)
- added R93: 0R, Resistor_SMD:R_0603_1608Metric, F.Cu at (64.0, 53.0)
- added R94: 0R, Resistor_SMD:R_0603_1608Metric, F.Cu at (70.0, 50.5)
- added U10: TXB0104RUT, Package_DFN_QFN:Texas_R-PUQFN-N12, F.Cu at (162.1, 66.1)
- added U11: TPS76333, Package_TO_SOT_SMD:SOT-23-5, F.Cu at (161.5, 82.7)
- added U12: TXB0104RUT, Package_DFN_QFN:Texas_R-PUQFN-N12, F.Cu at (161.6, 107.2)
- added U13: TXB0104RUT, Package_DFN_QFN:Texas_R-PUQFN-N12, F.Cu at (161.9, 100.9)
- added U14: TPS76333, Package_TO_SOT_SMD:SOT-23-5, F.Cu at (161.2, 117.5)
- added U6: TXB0104RUT, Package_DFN_QFN:Texas_R-PUQFN-N12, F.Cu at (109.3, 115.3)
- added U7: TXB0104RUT, Package_DFN_QFN:Texas_R-PUQFN-N12, F.Cu at (109.0, 121.6)
- added U8: TPS76333, Package_TO_SOT_SMD:SOT-23-5, F.Cu at (109.7, 105.0)
- added U9: TXB0104RUT, Package_DFN_QFN:Texas_R-PUQFN-N12, F.Cu at (161.9, 72.4)
- moved H2 91.6 mm to (137.6, 123.7)
- moved H1 10.6 mm to (137.6, 40.3)
- moved R18 8.51 mm to (107.3, 84.7), turned to 180 degrees
- moved R13 7.63 mm to (107.5, 77.5)
- moved R14 7.56 mm to (107.5, 76.7)
- moved R19 6.85 mm to (107.3, 83.8), turned to 180 degrees
- moved R20 3.93 mm to (107.5, 75.8), turned to 180 degrees
- moved R16 3.77 mm to (107.5, 78.3), turned to 180 degrees
- moved C13 2.96 mm to (111.7, 82.5)
- moved C14 2.96 mm to (109.7, 81.6)
- moved U5 2.96 mm to (109.6, 83.4)
- moved R15 2.96 mm to (107.3, 83.0)
- moved R17 2.96 mm to (107.3, 82.1)
- moved C11 2.92 mm to (112.0, 76.0)
- moved C12 2.92 mm to (110.0, 75.2), turned to 0 degrees
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Connections:
- J17 pad 1: unconnected-(J17-Pin_1-Pad1) -> /GP_SUB2/TP16_Pin16
- J17 pad 2: unconnected-(J17-Pin_2-Pad2) -> /GP_SUB2/TP6_Pin7
- J17 pad 22: unconnected-(J17-Pin_22-Pad22) -> /GP_SUB3/TP16_Pin16
- J17 pad 23: unconnected-(J17-Pin_23-Pad23) -> /GP_SUB3/TP6_Pin7
- J17 pad 24: unconnected-(J17-Pin_24-Pad24) -> /GP_SUB3/TP12_Pin8
- J17 pad 25: unconnected-(J17-Pin_25-Pad25) -> /GP_SUB3/TP13_Pin9
- J17 pad 26: unconnected-(J17-Pin_26-Pad26) -> /GP_SUB3/TP7_Pin11
- J17 pad 27: unconnected-(J17-Pin_27-Pad27) -> /GP_SUB3/TP15_Pin12
- J17 pad 28: unconnected-(J17-Pin_28-Pad28) -> /GP_SUB3/TP8_Pin13
- J17 pad 29: unconnected-(J17-Pin_29-Pad29) -> /GP_SUB3/TP2_Pin14
- J17 pad 3: unconnected-(J17-Pin_3-Pad3) -> /GP_SUB2/TP12_Pin8
- J17 pad 30: unconnected-(J17-Pin_30-Pad30) -> /GP_SUB3/GP_EN
- J17 pad 4: unconnected-(J17-Pin_4-Pad4) -> /GP_SUB2/TP13_Pin9
- J17 pad 5: unconnected-(J17-Pin_5-Pad5) -> /GP_SUB2/TP7_Pin11
- J17 pad 6: unconnected-(J17-Pin_6-Pad6) -> /GP_SUB2/TP15_Pin12
- J17 pad 7: unconnected-(J17-Pin_7-Pad7) -> /GP_SUB2/TP8_Pin13
- J17 pad 8: unconnected-(J17-Pin_8-Pad8) -> /GP_SUB2/TP2_Pin14
- J17 pad 9: unconnected-(J17-Pin_9-Pad9) -> /GP_SUB2/GP_EN
- J4 pad 22: unconnected-(J4-Pin_22-Pad22) -> /GP_SUB1/TP16_Pin16
- J4 pad 23: unconnected-(J4-Pin_23-Pad23) -> /GP_SUB1/TP6_Pin7
- J4 pad 24: unconnected-(J4-Pin_24-Pad24) -> /GP_SUB1/TP12_Pin8
- J4 pad 25: unconnected-(J4-Pin_25-Pad25) -> /GP_SUB1/TP13_Pin9
- J4 pad 26: unconnected-(J4-Pin_26-Pad26) -> /GP_SUB1/TP7_Pin11
- J4 pad 27: unconnected-(J4-Pin_27-Pad27) -> /GP_SUB1/TP15_Pin12
- J4 pad 28: unconnected-(J4-Pin_28-Pad28) -> /GP_SUB1/TP8_Pin13
- J4 pad 29: unconnected-(J4-Pin_29-Pad29) -> /GP_SUB1/TP2_Pin14
- J4 pad 30: unconnected-(J4-Pin_30-Pad30) -> /GP_SUB1/GP_EN
- R13 pad 1: Net-(U5-A4) -> Net-(U2-A3)
- R14 pad 1: Net-(U5-A3) -> Net-(U2-A2)
- R18 pad 1: Net-(U2-A3) -> Net-(U5-A4)
- R19 pad 1: Net-(U2-A2) -> Net-(U5-A3)
- R9 pad 1: GP1_EN -> PROT_EN
- U2 pad 8: /GP_SUB/TP12_Pin8 -> /GP_SUB/TP15_Pin12
- U2 pad 9: /GP_SUB/TP8_Pin13 -> /GP_SUB/TP16_Pin16
- U5 pad 7: /GP_SUB/TP15_Pin12 -> /GP_SUB/TP12_Pin8
- U5 pad 8: /GP_SUB/TP16_Pin16 -> /GP_SUB/TP8_Pin13
Routing:
- net VBUS: track 37.3 -> 331.3 mm, vias 13 -> 37
- net GND: track 11.9 -> 77.5 mm, vias 4 -> 45
- net P3V3_LOCAL: track 3.26 -> 51.0 mm, vias 0 -> 16
- net /GP_SUB3/P8: track 0.00 -> 36.9 mm
- net /GP_SUB1/P8: track 0.00 -> 36.9 mm
- net /GP_SUB2/P8: track 0.00 -> 36.9 mm
- net /GP_SUB1/P9: track 0.00 -> 36.5 mm
- net /GP_SUB3/P9: track 0.00 -> 36.5 mm
- net /GP_SUB2/P9: track 0.00 -> 36.5 mm
- net /GP_SUB3/P13: track 0.00 -> 29.4 mm
- net /GP_SUB2/P13: track 0.00 -> 29.4 mm
- net /GP_SUB1/P13: track 0.00 -> 29.4 mm
- net /GP_SUB2/P16: track 0.00 -> 28.3 mm
- net /GP_SUB1/P16: track 0.00 -> 28.3 mm
- net /GP_SUB3/P16: track 0.00 -> 28.3 mm
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- added copper zone on In2.Cu, net P3V3_LOCAL
