File: MCU.kicad_sch (KiCad schematic)
At the start: 32 parts, among them J1 F31L-1A7H1-11030, J17 Conn_02x30_Counter_Clockwise, J2 F31L-1A7H1-11030, J3 F31L-1A7H1-11030, J4 Conn_02x30_Counter_Clockwise, J6 Conn_01x02, U3 TPS76333, U4 TPS76333

Commit message: Add files via upload
Parts:
- added R89, R90: 1R, Resistor_SMD:R_0603_1608Metric, symbol Device:R_Small
Connections:
- net HMI_EN: now also R90.2
- net VBUS: now also R89.1, R90.1
- net GP_SUB1/TP16_Pin16: now reaches J4.22 (Pin_22)
- net GP_SUB1/TP6_Pin7: now reaches J4.23 (Pin_23)
- net GP_SUB1/TP12_Pin8: now reaches J4.24 (Pin_24)
- net GP_SUB1/TP13_Pin9: now reaches J4.25 (Pin_25)
- net GP_SUB1/TP7_Pin11: now reaches J4.26 (Pin_26)
- net GP_SUB1/TP15_Pin12: now reaches J4.27 (Pin_27)
- net GP_SUB1/TP8_Pin13: now reaches J4.28 (Pin_28)
- net GP_SUB1/TP2_Pin14: now reaches J4.29 (Pin_29)
- net GP_SUB1/GP_EN: now reaches J4.30 (Pin_30)
- net GP_SUB2/TP16_Pin16: now reaches J17.1 (Pin_1)
- net GP_SUB2/TP6_Pin7: now reaches J17.2 (Pin_2)
- net GP_SUB3/TP16_Pin16: now reaches J17.22 (Pin_22)
- net GP_SUB3/TP6_Pin7: now reaches J17.23 (Pin_23)
- net GP_SUB3/TP12_Pin8: now reaches J17.24 (Pin_24)
- net GP_SUB3/TP13_Pin9: now reaches J17.25 (Pin_25)
- net GP_SUB3/TP7_Pin11: now reaches J17.26 (Pin_26)
- net GP_SUB3/TP15_Pin12: now reaches J17.27 (Pin_27)
- net GP_SUB3/TP8_Pin13: now reaches J17.28 (Pin_28)
- net GP_SUB3/TP2_Pin14: now reaches J17.29 (Pin_29)
- net GP_SUB2/TP12_Pin8: now reaches J17.3 (Pin_3)
- net GP_SUB3/GP_EN: now reaches J17.30 (Pin_30)
- net GP_SUB2/TP13_Pin9: now reaches J17.4 (Pin_4)
- net GP_SUB2/TP7_Pin11: now reaches J17.5 (Pin_5)
- net GP_SUB2/TP15_Pin12: now reaches J17.6 (Pin_6)
- net GP_SUB2/TP8_Pin13: now reaches J17.7 (Pin_7)
- net GP_SUB2/TP2_Pin14: now reaches J17.8 (Pin_8)
- net GP_SUB2/GP_EN: now reaches J17.9 (Pin_9)
- net GP1_EN renamed PROT_EN
- net PROT_EN: now also R89.2
Other:
- added sheet GP_SUB1 (GP_SUB.kicad_sch)
- added sheet GP_SUB2 (GP_SUB.kicad_sch)
- added sheet GP_SUB3 (GP_SUB.kicad_sch)
- moved on the sheet: J17
