File: MCU.kicad_sch (KiCad schematic)
At the start: 34 parts, among them J1 F31L-1A7H1-11030, J17 Conn_02x30_Counter_Clockwise, J2 F31L-1A7H1-11030, J3 F31L-1A7H1-11030, J4 Conn_02x30_Counter_Clockwise, J6 Conn_01x02, U3 TPS76333, U4 TPS76333

Commit message: Add files via upload
Parts:
- added H5: MountingHole_Pad, MountingHole:MountingHole_2.2mm_M2_DIN965_Pad, symbol Mechanical:MountingHole_Pad
- added J22: Conn_01x02, Connector_PinHeader_2.54mm:PinHeader_1x02_P2.54mm_Vertical, symbol Connector_Generic:Conn_01x02
Connections:
- net BRSW_CTL_C: now also J4.33 (Pin_33)
- net GND: now also J17.10 (Pin_10), J17.11 (Pin_11), J17.12 (Pin_12), J17.13 (Pin_13), J17.14 (Pin_14), J17.15 (Pin_15), J17.16 (Pin_16), J17.17 (Pin_17), J17.18 (Pin_18), J17.19 (Pin_19), J17.20 (Pin_20), J17.21 (Pin_21), J17.43 (Pin_43), J17.44 (Pin_44), J17.45 (Pin_45), J17.46 (Pin_46), J17.47 (Pin_47), J17.48 (Pin_48), J17.49 (Pin_49), J17.50 (Pin_50), J17.51 (Pin_51), J17.52 (Pin_52), J17.53 (Pin_53), J17.54 (Pin_54), J17.55 (Pin_55), J17.56 (Pin_56), J17.57 (Pin_57), J17.58 (Pin_58), J17.59 (Pin_59), J17.60 (Pin_60), J4.10 (Pin_10), J4.11 (Pin_11), J4.12 (Pin_12), J4.13 (Pin_13), J4.14 (Pin_14), J4.15 (Pin_15), J4.16 (Pin_16), J4.17 (Pin_17), J4.18 (Pin_18), J4.19 (Pin_19), J4.20 (Pin_20), J4.21 (Pin_21), J4.22 (Pin_22), J4.23 (Pin_23), J4.24 (Pin_24), J4.25 (Pin_25), J4.26 (Pin_26), J4.27 (Pin_27), J4.28 (Pin_28), J4.29 (Pin_29), J4.30 (Pin_30), J4.42 (Pin_42), J4.43 (Pin_43), J4.44 (Pin_44), J4.45 (Pin_45), J4.46 (Pin_46), J4.47 (Pin_47), J4.48 (Pin_48), J4.49 (Pin_49), J4.50 (Pin_50), J4.51 (Pin_51), H5.1, J22.1 (Pin_1), J22.2 (Pin_2)
- net GP_SUB1/GP_EN: now also J4.52 (Pin_52); no longer J4.30 (Pin_30)
- net GP_SUB1/TP12_Pin8: now also J4.58 (Pin_58); no longer J4.24 (Pin_24)
- net GP_SUB1/TP13_Pin9: now also J4.57 (Pin_57); no longer J4.25 (Pin_25)
- net GP_SUB1/TP15_Pin12: now also J4.55 (Pin_55); no longer J4.27 (Pin_27)
- net GP_SUB1/TP16_Pin16: now also J4.60 (Pin_60); no longer J4.22 (Pin_22)
- net GP_SUB1/TP2_Pin14: now also J4.53 (Pin_53); no longer J4.29 (Pin_29)
- net GP_SUB1/TP6_Pin7: now also J4.59 (Pin_59); no longer J4.23 (Pin_23)
- net GP_SUB1/TP7_Pin11: now also J4.56 (Pin_56); no longer J4.26 (Pin_26)
- net GP_SUB1/TP8_Pin13: now also J4.54 (Pin_54); no longer J4.28 (Pin_28)
- net HMI_EN: now also J17.31 (Pin_31)
- net PA0_ADCIN5: now also J17.41 (Pin_41)
- net PA1_ADCIN6: now also J17.42 (Pin_42)
- net PA2_ADCIN7: now also J17.35 (Pin_35)
- net PA3_ADCIN8: now also J17.36 (Pin_36)
- net PB0_ADCIN15: now also J17.37 (Pin_37)
- net PB10_I2C2_SCL: now also J4.36 (Pin_36)
- net PB11_I2C2_SDA: now also J4.37 (Pin_37)
- net PC13_EXTI13: now also J4.31 (Pin_31)
- net PC1_ADCIN2: now also J17.38 (Pin_38)
- net PC2_ADCIN3: now also J17.39 (Pin_39)
- net PC3_ADCIN4: now also J17.40 (Pin_40)
- net PD10: now also J17.34 (Pin_34)
- net PD11: now also J17.33 (Pin_33)
- net PD13: now also J4.34 (Pin_34)
- net PD14: now also J4.40 (Pin_40)
- net PE10_EXTI10: now also J4.39 (Pin_39)
- net PE2: now also J4.41 (Pin_41)
- net PE3_TIM3_CH1: now also J4.35 (Pin_35)
- net PE5_EXTI5: now also J4.32 (Pin_32)
- net PE6_EXTI6: now also J4.38 (Pin_38)
- net PROT_EN: now also J17.32 (Pin_32)
Other:
- moved on the sheet: H1, H2, H3, H4, J17, J4

Commit message: Rails alim + libs
Parts:
- removed C10, C3, C5: 100nF, Capacitor_SMD:C_0402_1005Metric, symbol Device:C_Small
- removed C4: 4.7uF, Capacitor_SMD:C_0402_1005Metric, symbol Device:C_Small
- removed C6, C8: 1uF, Capacitor_SMD:C_0603_1608Metric, symbol Device:C_Small
- removed C7, C9: 4.7uF, Capacitor_SMD:C_0603_1608Metric, symbol Device:C_Small
- removed D1, D3: LED, LED_SMD:LED_0805_2012Metric, symbol Device:LED
- removed J1, J2, J3: F31L-1A7H1-11030, F31L-1A7H1-11030:AMPHENOL_F31L-1A7H1-11030, symbol F31L-1A7H1-11030:F31L-1A7H1-11030
- removed R10, R5: 9k1, Resistor_SMD:R_0603_1608Metric, symbol Device:R_Small
- removed R11, R6, R89, R90: 1R, Resistor_SMD:R_0603_1608Metric, symbol Device:R_Small
- removed R12, R7: 1k, Resistor_SMD:R_0603_1608Metric, symbol Device:R_Small
- removed R4, R9: 4k7, Resistor_SMD:R_0603_1608Metric, symbol Device:R_Small
- removed U3, U4: TPS76333, Package_TO_SOT_SMD:SOT-23-5, symbol Regulator_Linear:TPS76333
- added J1: HSEC8-150-01-X-RA-X, kicad_jlcpcb_hil_mcu_ep2:SAMTEC_HSEC8-150-01-X-RA-X, symbol HSEC8-150-01-X-RA-X:HSEC8-150-01-X-RA-X
- added J2: Barrel_Jack_MountingPin, Connector_BarrelJack:BarrelJack_CUI_PJ-063AH_Horizontal, symbol Connector:Barrel_Jack_MountingPin
- added U3: LMR36510ADDA, Package_SO:Texas_HTSOP-8-1EP_3.9x4.9mm_P1.27mm_EP2.95x4.9mm_Mask2.4x3.1mm_ThermalVias, symbol Regulator_Switching:LMR36510ADDA
Connections:
- net GND: now also J1.05, J1.06, J1.09, J1.11, J1.12, J1.17, J1.18, J1.23, J1.24, J1.27, J1.30, J1.33, J1.39, J1.40, J1.45, J1.46, J1.51, J1.52, J1.57, J1.58, J1.63, J1.64, J1.67, J1.70, J1.76, J1.77, J1.82, J1.89, J1.90, J1.95, J1.96
- net BRSW_CTL_C renamed ISOSW_OF_ST
- net ISOSW_OF_ST: now also J1.42
- net HMI_EN: no longer names the net of J17.31 (Pin_31)
- net PA0_ADCIN5 renamed V_US
- net V_US: now also J1.31
- net PA1_ADCIN6 renamed LEM_US_IN
- net LEM_US_IN: now also J1.92
- net PA2_ADCIN7 renamed SDMOS
- net SDMOS: now also J1.26
- net PA3_ADCIN8 renamed LEM_DS_IN
- net LEM_DS_IN: now also J1.86
- net PB0_ADCIN15 renamed V_CTANK
- net V_CTANK: now also J1.60
- net PB10_I2C2_SCL: no longer names the net of J4.36 (Pin_36)
- net PB11_I2C2_SDA renamed VPS_P24V_PG
- net VPS_P24V_PG: now also J1.34
- net PC13_EXTI13 renamed EN_PS_ACT
- net EN_PS_ACT: now also J1.47
- net PC1_ADCIN2 renamed V_HERMES
- net V_HERMES: now also J1.93
- net PC2_ADCIN3 renamed V_ACT
- net V_ACT: now also J1.66
- net PC3_ADCIN4 renamed V_DS
- net V_DS: now also J1.37
- net PD10 renamed ISOSW_HOLD_CMD
- net ISOSW_HOLD_CMD: now also J1.50
- net PD11: no longer names the net of J17.33 (Pin_33)
- net PD13 renamed PADLOCK_OF
- net PADLOCK_OF: now also J1.48
- net PD14 renamed SSR_CTL
- net SSR_CTL: now also J1.41
- net PE2 renamed ISOSW_INRUSH_CMD
- net ISOSW_INRUSH_CMD: now also J1.44
- net PE3_TIM3_CH1: no longer names the net of J4.35 (Pin_35)
- net PE5_EXTI5 renamed CTANK_CH_DISCH
- net CTANK_CH_DISCH: now also J1.83
- net PE6_EXTI6 renamed BTN_TRIP_TEST
- net BTN_TRIP_TEST: now also J1.20
- net PROT_EN: no longer names the net of J17.32 (Pin_32)
- new net DS_MISO: J1.21
- new net DS_MOSI: J1.19
- new net DS_NCS_C1: J1.15
- new net DS_NCS_C2: J1.13
- new net DS_SCLK: J1.25
- new net NEG10VAN: J1.100, J1.98
- new net OPCL_DS: J1.14
- new net OPCL_US: J1.61
- new net P24V: J1.53, J1.54, J1.55, J1.56, J2.1
- new net P3V7: J1.02, J1.04
- new net P5V: J1.01, J1.03, J1.97, J1.99, U3.8 (SW)
- new net US_MISO: J1.69
- new net US_MOSI: J1.71
- new net US_NCS_C1: J1.73
- new net US_NCS_C2: J1.75
- new net US_SCLK: J1.65
Other:
- sheet GP_SUB ports: added SDMOS; removed SD_MOS
- sheet GP_SUB1 ports: added SDMOS; removed SD_MOS
- sheet GP_SUB2 ports: added SDMOS; removed SD_MOS
- sheet GP_SUB3 ports: added SDMOS; removed SD_MOS
- note added: "LMR36520ADDAR"
- moved on the sheet: C16, C17, J6

Commit message: Power
Parts:
- removed C17: 100nF, Capacitor_SMD:C_0402_1005Metric, symbol Device:C_Small
- added C3: 1uF, Capacitor_SMD:C_0603_1608Metric, symbol Device:C_Small
- added C35: 18pF, Capacitor_SMD:C_0402_1005Metric, symbol Device:C_Small
- added C36: 100nF, Capacitor_SMD:C_0603_1608Metric, symbol Device:C_Small
- added C37: 18pF, Capacitor_SMD:C_0603_1608Metric, symbol Device:C_Small
- added C4: 10uF, Capacitor_SMD:C_0603_1608Metric, symbol Device:C_Small
- added C5, C6: 22uF, Capacitor_SMD:C_0603_1608Metric, symbol Device:C_Small
- added L1: 22uH, Inductor_SMD:L_TDK_SLF10145, symbol Device:L_Small
- added R89: 25.5k, Resistor_SMD:R_0603_1608Metric, symbol Device:R_Small
- added R90: 102k, Resistor_SMD:R_0603_1608Metric, symbol Device:R_Small
- added R95: 33k, Resistor_SMD:R_0603_1608Metric, symbol Device:R_Small
- added R96: 499k, Resistor_SMD:R_0603_1608Metric, symbol Device:R_Small
- added R97: 10k, Resistor_SMD:R_0603_1608Metric, symbol Device:R_Small
- added R98: 15k, Resistor_SMD:R_0603_1608Metric, symbol Device:R_Small
- C16: value 4.7uF -> 100nF; footprint Capacitor_SMD:C_0402_1005Metric -> Capacitor_SMD:C_0603_1608Metric; JLCPCB Part # C23733 -> (none); JLCPCB Part# (none) -> C1525
Connections:
- net NEG10VAN is gone; now on net GND: J1.100, J1.98
- net VBUS is gone; now on net P24V: C16.1, J6.1 (Pin_1)
- net GND: now also J2.2, J2.MP (MountPin), U3.1 (PGND), U3.9 (PAD), C3.2, C35.2, C4.2, C5.2, C6.2, R89.1, R95.1, R98.1
- net P24V: now also U3.2 (VIN), C4.1, R96.2
- net at U3.3 (EN): now also C35.1, R95.2, R96.1
- net at U3.4 (PG): now also R97.1, R98.2
- net at U3.5 (FB): now also C37.1, R89.2, R90.1
- net at U3.6 (VCC): now also C3.1
- net at U3.7 (BOOT): now also C36.1
- net P3V7 renamed P5VAN
- net P5VAN: now also J1.01, J1.03, J1.97, J1.99, C37.2, C5.1, C6.1, L1.2, R90.2, R97.2
- removed net P5V: J1.01, J1.03, J1.97, J1.99, U3.8 (SW)
- new net: C36.2, L1.1, U3.8 (SW)
- no-connect marks 5 -> 0
Other:
- added sheet Power (Power.kicad_sch)
- note removed: "HMI"
- note removed: "MainPWR"
- note removed: "PSU"
- moved on the sheet: J2, J6

Commit message: Ready for review
Parts:
- added H6: MountingHole_Pad, MountingHole:MountingHole_2.2mm_M2_DIN965_Pad, symbol Mechanical:MountingHole_Pad
- added J23: Conn_01x02, Connector_PinHeader_2.54mm:PinHeader_1x02_P2.54mm_Vertical, symbol Connector_Generic:Conn_01x02
Connections:
- net GND: now also J1.16, J1.28, J1.29, J1.35, J1.59, J1.62, J1.68, J1.74, J1.78, J1.88, J1.91, J1.94, H6.1
- net P5VAN: now also J23.1 (Pin_1)
- net PADLOCK_OF: now also J23.2 (Pin_2)
- net BTN_TRIP_TEST: no longer names the net of J1.20
- net BTN_TRIP_TEST: no longer J4.38 (Pin_38)
Other:
- removed sheet Power

Commit message: For review
Parts:
- added TP1: TestPoint, TestPoint:TestPoint_Pad_1.5x1.5mm, symbol Connector:TestPoint
Connections:
- net at R97.1, R98.2, U3.4 (PG): now also TP1.1
Other:
- note added: "GROUND"
- note added: "GoldFinger"
- note added: "P24V → 5V"
- note added: "PADLOCK SIMU"
- note added: "Power Nets labels"
- note added: "VIN"
- moved on the sheet: C16, C3, C35, C36, C37, C4, C5, C6, H1, H2, H3, H4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

Commit message: Refactor GreenPak Pinout
Connections:
- no-connect marks 0 -> 17
Changed lines of the file:
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@@
 		(color 0 0 0 0)
+	)
+	(no_connect
+		(at 193.04 58.42)
+	)
+	(no_connect
+		(at 167.64 76.2)
+	)
+	(no_connect
+		(at 167.64 78.74)
+	)
+	(no_connect
+		(at 116.84 83.82)
+	)
+	(no_connect
+		(at 116.84 63.5)
+	)
+	(no_connect
+		(at 116.84 81.28)
+	)
+	(no_connect
+		(at 116.84 60.96)
+	)
+	(no_connect
+		(at 116.84 45.72)
+	)
+	(no_connect
+		(at 91.44 45.72)
+	)
+	(no_connect
+		(at 167.64 71.12)
+	)
+	(no_connect
+		(at 116.84 48.26)
+	)
+	(no_connect
+		(at 193.04 73.66)
+	)
+	(no_connect
+		(at 91.44 99.06)
+	)
+	(no_connect
+		(at 193.04 68.58)
+	)
+	(no_connect
+		(at 167.64 68.58)
+	)
+	(no_connect
+		(at 116.84 76.2)
+	)
+	(no_connect
+		(at 91.44 91.44)
 	)
 	(wire

Commit message: OPCL via LevelShifters
Other:
- sheet GP_SUB ports: added none; removed SDMOS
- sheet GP_SUB1 ports: added none; removed SDMOS
- sheet GP_SUB2 ports: added none; removed SDMOS
- sheet GP_SUB3 ports: added none; removed SDMOS
Changed lines of the file:
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@@
 	(wire
 		(pts
-			(xy 33.02 209.55) (xy 41.275 209.55)
-		)
-		(stroke
-			(width 0)
-			(type default)
-		)
-	)
-	(wire
-		(pts
 			(xy 340.36 187.96) (xy 340.36 193.04)
 		)
@@
 	(wire
 		(pts
-			(xy 266.7 209.55) (xy 273.05 209.55)
-		)
-		(stroke
-			(width 0)
-			(type default)
-		)
-	)
-	(wire
-		(pts
-			(xy 247.65 262.89) (xy 254 262.89)
-		)
-		(stroke
-			(width 0)
-			(type default)
-		)
-	)
-	(wire
-		(pts
 			(xy 72.39 204.47) (xy 82.55 204.47)
 		)
@@
 	(wire
 		(pts
-			(xy 151.13 209.55) (xy 144.78 209.55)
-		)
-		(stroke
-			(width 0)
-			(type default)
-		)
-	)
-	(wire
-		(pts
 			(xy 203.2 209.55) (xy 234.95 209.55)
 		)
@@
 		)
 	)
-	(global_label "SDMOS"
-		(shape input)
-		(at 273.05 209.55 0)
-		(fields_autoplaced yes)
-		(effects
-			(font
-				(size 1.27 1.27)
-			)
-			(justify left)
-		)
-		(property "Intersheetrefs" "${INTERSHEET_REFS}"
-			(at 279.6033 209.55 0)
-			(hide yes)
-			(show_name no)
-			(do_not_autoplace no)
-			(effects
-				(font
-					(size 1.27 1.27)
-				)
-				(justify left)
-			)
-		)
-	)
 	(global_label "A0V"
 		(shape input)
@@
 		)
 	)
-	(global_label "SDMOS"
-		(shape input)
-		(at 33.02 209.55 180)
-		(fields_autoplaced yes)
-		(effects
-			(font
-				(size 1.27 1.27)
-			)
-			(justify right)
-		)
-		(property "Intersheetrefs" "${INTERSHEET_REFS}"
-			(at 23.5639 209.55 0)
-			(hide yes)
-			(show_name no)
-			(do_not_autoplace no)
-			(effects
-				(font
-					(size 1.27 1.27)
-				)
-				(justify right)
-			)
-		)
-	)
 	(global_label "A0V"
 		(shape input)
@@
 		)
 	)
-	(global_label "SDMOS"
-		(shape input)
-		(at 254 262.89 0)
-		(fields_autoplaced yes)
-		(effects
-			(font
-				(size 1.27 1.27)
-			)
-			(justify left)
-		)
-		(property "Intersheetrefs" "${INTERSHEET_REFS}"
-			(at 260.5533 262.89 0)
-			(hide yes)
-			(show_name no)
-			(do_not_autoplace no)
-			(effects
-				(font
-					(size 1.27 1.27)
-				)
-				(justify left)
-			)
-		)
-	)
 	(global_label "DS_MOSI"
 		(shape input)
@@
 		)
 	)
-	(global_label "SDMOS"
-		(shape input)
-		(at 151.13 209.55 0)
-		(fields_autoplaced yes)
-		(effects
-			(font
-				(size 1.27 1.27)
-			)
-			(justify left)
-		)
-		(property "Intersheetrefs" "${INTERSHEET_REFS}"
-			(at 157.6833 209.55 0)
-			(hide yes)
-			(show_name no)
-			(do_not_autoplace no)
-			(effects
-				(font
-					(size 1.27 1.27)
-				)
-				(justify left)
-			)
-		)
-	)
 	(global_label "V_CTANK"
 		(shape input)
@@
 			)
 		)
-		(pin "SDMOS" input
-			(at 266.7 209.55 0)
-			(effects
-				(font
-					(size 1.27 1.27)
-				)
-				(justify right)
-			)
-		)
 		(pin "MOS_TRIP" input
 			(at 266.7 213.36 0)
@@
 			)
 		)
-		(pin "SDMOS" input
-			(at 41.275 209.55 180)
-			(effects
-				(font
-					(size 1.27 1.27)
-				)
-				(justify left)
-			)
-		)
 		(pin "MOS_TRIP" input
 			(at 41.275 213.36 180)
@@
 			)
 		)
-		(pin "SDMOS" input
-			(at 247.65 262.89 0)
-			(effects
-				(font
-					(size 1.27 1.27)
-				)
-				(justify right)
-			)
-		)
 		(pin "MOS_TRIP" input
 			(at 247.65 266.7 0)
@@
 			(effects
 				(font
-					(size 1.27 1.27)
-				)
-				(justify right)
-			)
-		)
-		(pin "SDMOS" input
-			(at 144.78 209.55 0)
-			(effects
-				(font
